File: hardware/kicad/hoermann-hcp-adapter.kicad_sch (KiCad schematic)
At the start: 5 parts, among them J1 HCP2 6P6C unshielded, AliExpr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, U1 ESP32-C3 Super Mini, U2 Isolated auto-direction RS485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

Commit message: Compact PCB layout with real module footprints
Shrink the board to 63 x 42 mm, put the RJ12 jack at the edge and
replace the placeholder footprints with a project library: KiCad's
Amphenol 54601 footprint for the 95001-type jack, and LM2596 HW-411,
isolated RS485 and ESP32-C3 Super Mini footprints measured from vendor
material. Mounting uses the LM2596 module holes plus one hole under the
ESP32. pcb.py now instantiates library footprints, checks routes against
pad positions and runs DRC; the schematic assigns the same footprints.

Co-Authored-By: Claude Fable 5.1 <noreply@anthropic.com>
Parts:
- J1: footprint : -> HCP:RJ12_Amphenol_54601-x06_Horizontal
- JP1: footprint : -> HCP:PinHeader_1x02_P2.54mm_Vertical
- PS1: footprint : -> HCP:LM2596_HW-411
- U1: footprint : -> HCP:ESP32-C3_SuperMini
- U2: footprint : -> HCP:RS485_Isolated_34x18
Changed lines of the file:
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@@
           (size 1.27 1.27))
         (justify left)))
-    (property "Footprint" ":"
+    (property "Footprint" "HCP:RJ12_Amphenol_54601-x06_Horizontal"
       (at 75.00 105.00 0)
       (effects
@@
     (instances
       (project "SKiDL-Generated"
-        (path "/a35db754-4ccf-47c2-b339-0bbc1bfc557f"
+        (path "/dd2e1869-6021-4073-8001-80164229c12d"
           (reference "J1")
           (unit 1)))))
@@
           (size 1.27 1.27))
         (justify left)))
-    (property "Footprint" ":"
+    (property "Footprint" "HCP:LM2596_HW-411"
       (at 105.00 60.00 0)
       (effects
@@
     (instances
       (project "SKiDL-Generated"
-        (path "/a35db754-4ccf-47c2-b339-0bbc1bfc557f"
+        (path "/dd2e1869-6021-4073-8001-80164229c12d"
           (reference "PS1")
           (unit 1)))))
@@
           (size 1.27 1.27))
         (justify left)))
-    (property "Footprint" ":"
+    (property "Footprint" "HCP:PinHeader_1x02_P2.54mm_Vertical"
       (at 145.00 60.00 0)
       (effects
@@
     (instances
       (project "SKiDL-Generated"
-        (path "/a35db754-4ccf-47c2-b339-0bbc1bfc557f"
+        (path "/dd2e1869-6021-4073-8001-80164229c12d"
           (reference "JP1")
           (unit 1)))))
@@
           (size 1.27 1.27))
         (justify left)))
-    (property "Footprint" ":"
+    (property "Footprint" "HCP:ESP32-C3_SuperMini"
       (at 150.00 105.00 0)
       (effects
@@
     (instances
       (project "SKiDL-Generated"
-        (path "/a35db754-4ccf-47c2-b339-0bbc1bfc557f"
+        (path "/dd2e1869-6021-4073-8001-80164229c12d"
           (reference "U1")
           (unit 1)))))
@@
           (size 1.27 1.27))
         (justify left)))
-    (property "Footprint" ":"
+    (property "Footprint" "HCP:RS485_Isolated_34x18"
       (at 110.00 105.00 0)
       (effects
@@
     (instances
       (project "SKiDL-Generated"
-        (path "/a35db754-4ccf-47c2-b339-0bbc1bfc557f"
+        (path "/dd2e1869-6021-4073-8001-80164229c12d"
           (reference "U2")
           (unit 1)))))
