File: hardware/pcb/generated/hcp.kicad_pcb (KiCad board)
At the start: 2 copper layers, 65 x 44.5 mm, 9 parts, among them J1 HCP2 6P6C, U1 ESP32-C3 Super Mini, U2 Isolated RS485

Commit message: Regenerate outputs
Co-Authored-By: Claude Fable 5.1 <noreply@anthropic.com>
Other:
- board text added: "Hörmann HCP2 Adapter afc2ea8"
- board text removed: "Hörmann HCP2 Adapter cabe87e"
Changed lines of the file:
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@@
   (via (at 154.5 103.27) (size 0.8) (drill 0.4) (layers "F.Cu" "B.Cu") (net 8))
   (gr_rect (start 116.0 68.0) (end 181.0 112.5) (stroke (width 0.1) (type default)) (fill none) (layer "Edge.Cuts"))
-  (gr_text "Hörmann HCP2 Adapter cabe87e" (at 145.5 92.0 0) (layer "F.SilkS") (effects (font (size 0.8 0.8) (thickness 0.15))))
+  (gr_text "Hörmann HCP2 Adapter afc2ea8" (at 145.5 92.0 0) (layer "F.SilkS") (effects (font (size 0.8 0.8) (thickness 0.15))))
   (gr_text "(C) 2026" (at 126.6 84.0 0) (layer "F.SilkS") (effects (font (size 0.8 0.8) (thickness 0.15))))
   (gr_text "Thies Gerken" (at 126.6 85.4 0) (layer "F.SilkS") (effects (font (size 0.8 0.8) (thickness 0.15))))

Commit message: Regenerate outputs
Co-Authored-By: Claude Fable 5.1 <noreply@anthropic.com>
Other:
- board text added: "3ae80be"
- board text added: "HCP2 Adapter"
- board text added: "Hörmann"
- board text removed: "Hörmann HCP2 Adapter afc2ea8"
Changed lines of the file:
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@@
     (descr "95001-type 6P6C modular jack, side entry, front face flush with the board edge. Pegs 2.4 mm at 12.0 mm, pins 1.02 mm stagger in rows 8.3/10.84 mm behind the edge. From vendor drawings, verify on delivered part.")
     (tags "RJ12 RJ11 6P6C 95001")
-    (property "Reference" "J1" (at 0.00 14.60 0) (layer "F.SilkS") (effects (font (size 1.0 1.0) (thickness 0.15))))
+    (property "Reference" "J1" (at 0.00 3.00 0) (layer "F.SilkS") (effects (font (size 1.0 1.0) (thickness 0.15))))
     (property "Value" "HCP2 6P6C" (at 0 16.0 0) (layer "F.Fab") (effects (font (size 1.0 1.0) (thickness 0.15))))
     (property "Datasheet" "" (at 0 0 0) (layer "F.Fab") (hide yes) (effects (font (size 1.0 1.0) (thickness 0.15))))
@@
   (via (at 154.5 103.27) (size 0.8) (drill 0.4) (layers "F.Cu" "B.Cu") (net 8))
   (gr_rect (start 116.0 68.0) (end 181.0 112.5) (stroke (width 0.1) (type default)) (fill none) (layer "Edge.Cuts"))
-  (gr_text "Hörmann HCP2 Adapter afc2ea8" (at 145.5 92.0 0) (layer "F.SilkS") (effects (font (size 0.8 0.8) (thickness 0.15))))
-  (gr_text "(C) 2026" (at 126.6 84.0 0) (layer "F.SilkS") (effects (font (size 0.8 0.8) (thickness 0.15))))
-  (gr_text "Thies Gerken" (at 126.6 85.4 0) (layer "F.SilkS") (effects (font (size 0.8 0.8) (thickness 0.15))))
+  (gr_text "Hörmann" (at 126.8 82.6 0) (layer "F.SilkS") (effects (font (size 0.8 0.8) (thickness 0.15))))
+  (gr_text "HCP2 Adapter" (at 126.8 84.0 0) (layer "F.SilkS") (effects (font (size 0.8 0.8) (thickness 0.15))))
+  (gr_text "3ae80be" (at 126.8 85.4 0) (layer "F.SilkS") (effects (font (size 0.8 0.8) (thickness 0.15))))
+  (gr_text "(C) 2026" (at 126.8 86.8 0) (layer "F.SilkS") (effects (font (size 0.8 0.8) (thickness 0.15))))
+  (gr_text "Thies Gerken" (at 126.8 88.2 0) (layer "F.SilkS") (effects (font (size 0.8 0.8) (thickness 0.15))))
   (gr_text "1" (at 122.45 80.6 0) (layer "F.SilkS") (effects (font (size 0.8 0.8) (thickness 0.15))))
   (gr_text "DISCONNECT" (at 178.4 87.2 90) (layer "F.SilkS") (effects (font (size 0.8 0.8) (thickness 0.15))))

Commit message: Regenerate outputs
Co-Authored-By: Claude Fable 5.1 <noreply@anthropic.com>
Parts:
- moved JP1 0.40 mm to (179.4, 76.0)
Other:
- board text added: "!"
- board text added: "8e51ebe"
- board text removed: "3ae80be"
Changed lines of the file:
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@@
   (footprint "HCP:PinHeader_1x02_P2.54mm_Vertical"
   	(layer "F.Cu")
-    (at 179.0 76.0 0)
+    (at 179.4 76.0 0)
   	(descr "Through hole straight pin header, 1x02, 2.54mm pitch, single row")
   	(tags "Through hole pin header THT 1x02 2.54mm single row")
   	(property "Reference" "JP1"
-  		(at 0.00 5.10 0)
+  		(at -2.00 1.27 90)
   		(layer "F.SilkS")
   		(effects
@@
   (segment (start 174.9 71.1) (end 174.9 74.2) (width 0.8) (layer "F.Cu") (net 5))
   (segment (start 174.9 74.2) (end 176.7 76.0) (width 0.8) (layer "F.Cu") (net 5))
-  (segment (start 176.7 76.0) (end 179.0 76.0) (width 0.8) (layer "F.Cu") (net 5))
-  (segment (start 179.0 78.54) (end 179.0 79.5) (width 0.8) (layer "B.Cu") (net 6))
-  (segment (start 179.0 79.5) (end 180.0 80.5) (width 0.8) (layer "B.Cu") (net 6))
-  (segment (start 180.0 80.5) (end 180.0 109.62) (width 0.8) (layer "B.Cu") (net 6))
+  (segment (start 176.7 76.0) (end 179.4 76.0) (width 0.8) (layer "F.Cu") (net 5))
+  (segment (start 179.4 78.54) (end 179.4 79.5) (width 0.8) (layer "B.Cu") (net 6))
+  (segment (start 179.4 79.5) (end 180.0 80.1) (width 0.8) (layer "B.Cu") (net 6))
+  (segment (start 180.0 80.1) (end 180.0 109.62) (width 0.8) (layer "B.Cu") (net 6))
   (segment (start 180.0 109.62) (end 178.29 109.62) (width 0.8) (layer "B.Cu") (net 6))
   (segment (start 173.21 109.62) (end 173.21 105.81) (width 0.5) (layer "F.Cu") (net 7))
@@
   (via (at 154.5 103.27) (size 0.8) (drill 0.4) (layers "F.Cu" "B.Cu") (net 8))
   (gr_rect (start 116.0 68.0) (end 181.0 112.5) (stroke (width 0.1) (type default)) (fill none) (layer "Edge.Cuts"))
+  (gr_line (start 179.0 83.3) (end 179.0 80.6) (stroke (width 0.2) (type default)) (layer "F.SilkS"))
+  (gr_line (start 179.0 80.6) (end 178.4 81.4) (stroke (width 0.2) (type default)) (layer "F.SilkS"))
+  (gr_line (start 179.0 80.6) (end 179.6 81.4) (stroke (width 0.2) (type default)) (layer "F.SilkS"))
   (gr_text "Hörmann" (at 126.8 82.6 0) (layer "F.SilkS") (effects (font (size 0.8 0.8) (thickness 0.15))))
   (gr_text "HCP2 Adapter" (at 126.8 84.0 0) (layer "F.SilkS") (effects (font (size 0.8 0.8) (thickness 0.15))))
-  (gr_text "3ae80be" (at 126.8 85.4 0) (layer "F.SilkS") (effects (font (size 0.8 0.8) (thickness 0.15))))
+  (gr_text "8e51ebe" (at 126.8 85.4 0) (layer "F.SilkS") (effects (font (size 0.8 0.8) (thickness 0.15))))
   (gr_text "(C) 2026" (at 126.8 86.8 0) (layer "F.SilkS") (effects (font (size 0.8 0.8) (thickness 0.15))))
   (gr_text "Thies Gerken" (at 126.8 88.2 0) (layer "F.SilkS") (effects (font (size 0.8 0.8) (thickness 0.15))))
   (gr_text "1" (at 122.45 80.6 0) (layer "F.SilkS") (effects (font (size 0.8 0.8) (thickness 0.15))))
-  (gr_text "DISCONNECT" (at 178.4 87.2 90) (layer "F.SilkS") (effects (font (size 0.8 0.8) (thickness 0.15))))
-  (gr_text "FOR USB" (at 179.6 87.2 90) (layer "F.SilkS") (effects (font (size 0.8 0.8) (thickness 0.15))))
+  (gr_text "!" (at 177.5 82.0 0) (layer "F.SilkS") (effects (font (size 1.4 1.4) (thickness 0.25))))
+  (gr_text "DISCONNECT" (at 178.4 88.2 90) (layer "F.SilkS") (effects (font (size 0.8 0.8) (thickness 0.15))))
+  (gr_text "FOR USB" (at 179.6 88.2 90) (layer "F.SilkS") (effects (font (size 0.8 0.8) (thickness 0.15))))
   (gr_text "ANT" (at 156.9 102.0 90) (layer "F.SilkS") (effects (font (size 0.8 0.8) (thickness 0.15))))
   (embedded_fonts no)

Commit message: Regenerate outputs
Co-Authored-By: Claude Fable 5.1 <noreply@anthropic.com>
Other:
- board text added: "5bc247c"
- board text removed: "8e51ebe"
Changed lines of the file:
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@@
     (layer "F.Cu")
     (at 154.45 80.25 0)
-    (descr "LM2596 HW-411 adjustable buck module, 43.5x21.5 mm, corner terminals, 2x M3 holes shared with carrier. Geometry from vendor photos, verify on delivered part.")
+    (descr "LM2596 HW-411 adjustable buck module, 43.4x21.2 mm, corner terminals 39.4x17.5 mm, 2x M3 holes 30.7x16.8 mm shared with carrier. Measured on delivered module.")
     (tags "LM2596 HW-411 buck module")
     (property "Reference" "PS1" (at 0.00 6.95 0) (layer "F.SilkS") (effects (font (size 1.0 1.0) (thickness 0.15))))
@@
     (property "Description" "" (at 0 0 0) (layer "F.Fab") (hide yes) (effects (font (size 1.0 1.0) (thickness 0.15))))
     (attr through_hole)
-    (fp_rect (start -21.75 -10.75) (end 21.75 10.75) (stroke (width 0.1) (type default)) (fill none) (layer "F.Fab"))
-    (fp_rect (start -21.9 -10.9) (end 21.9 10.9) (stroke (width 0.12) (type default)) (fill none) (layer "F.SilkS"))
-    (fp_rect (start -22.0 -11.0) (end 22.0 11.0) (stroke (width 0.05) (type default)) (fill none) (layer "F.CrtYd"))
-    (pad "1" thru_hole rect (at -20.45 -9.15) (size 2.4 2.4) (drill 1.1) (layers "*.Cu" "*.Mask") (remove_unused_layers no) (net 2 "HCP_25V"))
-    (fp_text user "IN+" (at -20.45 -11.15 0) (layer "F.Fab") (effects (font (size 0.7 0.7) (thickness 0.10))))
-    (pad "2" thru_hole circle (at -20.45 9.15) (size 2.4 2.4) (drill 1.1) (layers "*.Cu" "*.Mask") (remove_unused_layers no) (net 1 "HCP_GND"))
-    (fp_text user "IN-" (at -20.45 11.15 0) (layer "F.Fab") (effects (font (size 0.7 0.7) (thickness 0.10))))
-    (pad "3" thru_hole circle (at 20.45 -9.15) (size 2.4 2.4) (drill 1.1) (layers "*.Cu" "*.Mask") (remove_unused_layers no) (net 5 "BUCK_5V"))
-    (fp_text user "OUT+" (at 20.45 -11.15 0) (layer "F.Fab") (effects (font (size 0.7 0.7) (thickness 0.10))))
-    (pad "4" thru_hole circle (at 20.45 9.15) (size 2.4 2.4) (drill 1.1) (layers "*.Cu" "*.Mask") (remove_unused_layers no) (net 1 "HCP_GND"))
-    (fp_text user "OUT-" (at 20.45 11.15 0) (layer "F.Fab") (effects (font (size 0.7 0.7) (thickness 0.10))))
+    (fp_rect (start -21.7 -10.6) (end 21.7 10.6) (stroke (width 0.1) (type default)) (fill none) (layer "F.Fab"))
+    (fp_rect (start -21.849999999999998 -10.75) (end 21.849999999999998 10.75) (stroke (width 0.12) (type default)) (fill none) (layer "F.SilkS"))
+    (fp_rect (start -21.95 -10.85) (end 21.95 10.85) (stroke (width 0.05) (type default)) (fill none) (layer "F.CrtYd"))
+    (pad "1" thru_hole rect (at -19.7 -8.75) (size 2.4 2.4) (drill 1.1) (layers "*.Cu" "*.Mask") (remove_unused_layers no) (net 2 "HCP_25V"))
+    (fp_text user "IN+" (at -19.7 -10.75 0) (layer "F.Fab") (effects (font (size 0.7 0.7) (thickness 0.10))))
+    (pad "2" thru_hole circle (at -19.7 8.75) (size 2.4 2.4) (drill 1.1) (layers "*.Cu" "*.Mask") (remove_unused_layers no) (net 1 "HCP_GND"))
+    (fp_text user "IN-" (at -19.7 10.75 0) (layer "F.Fab") (effects (font (size 0.7 0.7) (thickness 0.10))))
+    (pad "3" thru_hole circle (at 19.7 -8.75) (size 2.4 2.4) (drill 1.1) (layers "*.Cu" "*.Mask") (remove_unused_layers no) (net 5 "BUCK_5V"))
+    (fp_text user "OUT+" (at 19.7 -10.75 0) (layer "F.Fab") (effects (font (size 0.7 0.7) (thickness 0.10))))
+    (pad "4" thru_hole circle (at 19.7 8.75) (size 2.4 2.4) (drill 1.1) (layers "*.Cu" "*.Mask") (remove_unused_layers no) (net 1 "HCP_GND"))
+    (fp_text user "OUT-" (at 19.7 10.75 0) (layer "F.Fab") (effects (font (size 0.7 0.7) (thickness 0.10))))
     (pad "" np_thru_hole circle (at -15.35 -8.4) (size 3.2 3.2) (drill 3.2) (layers "*.Cu" "*.Mask"))
     (pad "" np_thru_hole circle (at 15.35 8.4) (size 3.2 3.2) (drill 3.2) (layers "*.Cu" "*.Mask"))
@@
   (segment (start 127.55 77.6) (end 126.53 76.58) (width 0.5) (layer "F.Cu") (net 2))
   (segment (start 126.53 76.58) (end 126.53 76.3) (width 0.5) (layer "F.Cu") (net 2))
-  (segment (start 126.53 76.3) (end 126.53 71.1) (width 0.8) (layer "F.Cu") (net 2))
-  (segment (start 126.53 71.1) (end 134.0 71.1) (width 0.8) (layer "F.Cu") (net 2))
+  (segment (start 126.53 76.3) (end 126.53 71.5) (width 0.8) (layer "F.Cu") (net 2))
+  (segment (start 126.53 71.5) (end 134.75 71.5) (width 0.8) (layer "F.Cu") (net 2))
   (segment (start 122.45 76.3) (end 122.45 77.82) (width 0.5) (layer "B.Cu") (net 1))
   (segment (start 122.45 77.82) (end 123.47 78.84) (width 0.5) (layer "B.Cu") (net 1))
   (segment (start 123.47 78.84) (end 123.47 82.5) (width 0.8) (layer "B.Cu") (net 1))
-  (segment (start 123.47 82.5) (end 134.0 82.5) (width 0.8) (layer "B.Cu") (net 1))
-  (segment (start 134.0 82.5) (end 134.0 89.4) (width 0.8) (layer "B.Cu") (net 1))
-  (segment (start 134.0 89.4) (end 134.0 91.9) (width 0.8) (layer "F.Cu") (net 1))
-  (segment (start 134.0 91.9) (end 174.9 91.9) (width 0.8) (layer "F.Cu") (net 1))
-  (segment (start 174.9 91.9) (end 174.9 89.4) (width 0.8) (layer "F.Cu") (net 1))
-  (segment (start 174.9 91.9) (end 179.8 91.9) (width 0.5) (layer "F.Cu") (net 1))
+  (segment (start 123.47 82.5) (end 134.75 82.5) (width 0.8) (layer "B.Cu") (net 1))
+  (segment (start 134.75 82.5) (end 134.75 89.0) (width 0.8) (layer "B.Cu") (net 1))
+  (segment (start 134.75 89.0) (end 134.75 91.9) (width 0.8) (layer "F.Cu") (net 1))
+  (segment (start 134.75 91.9) (end 174.15 91.9) (width 0.8) (layer "F.Cu") (net 1))
+  (segment (start 174.15 91.9) (end 174.15 89.0) (width 0.8) (layer "F.Cu") (net 1))
+  (segment (start 174.15 91.9) (end 179.8 91.9) (width 0.5) (layer "F.Cu") (net 1))
   (segment (start 179.8 91.9) (end 179.8 111.2) (width 0.5) (layer "F.Cu") (net 1))
   (segment (start 179.8 111.2) (end 175.75 111.2) (width 0.5) (layer "F.Cu") (net 1))
@@
   (segment (start 155.5 91.9) (end 155.5 98.19) (width 0.5) (layer "F.Cu") (net 1))
   (segment (start 155.5 98.19) (end 152.5 98.19) (width 0.5) (layer "F.Cu") (net 1))
-  (segment (start 174.9 71.1) (end 174.9 74.2) (width 0.8) (layer "F.Cu") (net 5))
-  (segment (start 174.9 74.2) (end 176.7 76.0) (width 0.8) (layer "F.Cu") (net 5))
-  (segment (start 176.7 76.0) (end 179.4 76.0) (width 0.8) (layer "F.Cu") (net 5))
+  (segment (start 174.15 71.5) (end 174.15 74.2) (width 0.8) (layer "F.Cu") (net 5))
+  (segment (start 174.15 74.2) (end 175.95 76.0) (width 0.8) (layer "F.Cu") (net 5))
+  (segment (start 175.95 76.0) (end 179.4 76.0) (width 0.8) (layer "F.Cu") (net 5))
   (segment (start 179.4 78.54) (end 179.4 79.5) (width 0.8) (layer "B.Cu") (net 6))
   (segment (start 179.4 79.5) (end 180.0 80.1) (width 0.8) (layer "B.Cu") (net 6))
@@
   (gr_text "Hörmann" (at 126.8 82.6 0) (layer "F.SilkS") (effects (font (size 0.8 0.8) (thickness 0.15))))
   (gr_text "HCP2 Adapter" (at 126.8 84.0 0) (layer "F.SilkS") (effects (font (size 0.8 0.8) (thickness 0.15))))
-  (gr_text "8e51ebe" (at 126.8 85.4 0) (layer "F.SilkS") (effects (font (size 0.8 0.8) (thickness 0.15))))
+  (gr_text "5bc247c" (at 126.8 85.4 0) (layer "F.SilkS") (effects (font (size 0.8 0.8) (thickness 0.15))))
   (gr_text "(C) 2026" (at 126.8 86.8 0) (layer "F.SilkS") (effects (font (size 0.8 0.8) (thickness 0.15))))
   (gr_text "Thies Gerken" (at 126.8 88.2 0) (layer "F.SilkS") (effects (font (size 0.8 0.8) (thickness 0.15))))

Commit message: Regenerate outputs
Co-Authored-By: Claude Fable 5.1 <noreply@anthropic.com>
Routing:
- net HCP_B_MINUS: track 35.2 -> 28.1 mm
- net HCP_A_PLUS: track 35.2 -> 42.2 mm, vias 0 -> 1
- net HCP_25V: track 16.0 -> 15.0 mm
Other:
- board text added: "f21ee3d"
- board text removed: "5bc247c"
Changed lines of the file:
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@@
     (layer "F.Cu")
     (at 125.0 68.0 0)
-    (descr "95001-type 6P6C modular jack, side entry, front face flush with the board edge. Pegs 2.4 mm at 12.0 mm, pins 1.02 mm stagger in rows 8.3/10.84 mm behind the edge. From vendor drawings, verify on delivered part.")
+    (descr "95001-type 6P6C modular jack, side entry, front face flush with the board edge. Pegs 2.4 mm at 12.0 mm, pins 1.02 mm stagger in rows 8.3/10.84 mm behind the edge, odd pins in the rear row. From vendor drawings, verify on delivered part.")
     (tags "RJ12 RJ11 6P6C 95001")
     (property "Reference" "J1" (at 0.00 3.00 0) (layer "F.SilkS") (effects (font (size 1.0 1.0) (thickness 0.15))))
@@
     (property "Description" "" (at 0 0 0) (layer "F.Fab") (hide yes) (effects (font (size 1.0 1.0) (thickness 0.15))))
     (attr through_hole)
-    (pad "1" thru_hole rect (at -2.55 8.3) (size 1.6 1.6) (drill 1.0) (layers "*.Cu" "*.Mask") (remove_unused_layers no) (net 1 "HCP_GND"))
-    (pad "2" thru_hole circle (at -1.53 10.84) (size 1.6 1.6) (drill 1.0) (layers "*.Cu" "*.Mask") (remove_unused_layers no) (net 1 "HCP_GND"))
-    (pad "3" thru_hole circle (at -0.51 8.3) (size 1.6 1.6) (drill 1.0) (layers "*.Cu" "*.Mask") (remove_unused_layers no) (net 4 "HCP_B_MINUS"))
-    (pad "4" thru_hole circle (at 0.51 10.84) (size 1.6 1.6) (drill 1.0) (layers "*.Cu" "*.Mask") (remove_unused_layers no) (net 3 "HCP_A_PLUS"))
-    (pad "5" thru_hole circle (at 1.53 8.3) (size 1.6 1.6) (drill 1.0) (layers "*.Cu" "*.Mask") (remove_unused_layers no) (net 2 "HCP_25V"))
-    (pad "6" thru_hole circle (at 2.55 10.84) (size 1.6 1.6) (drill 1.0) (layers "*.Cu" "*.Mask") (remove_unused_layers no) (net 2 "HCP_25V"))
+    (pad "1" thru_hole rect (at -2.55 10.84) (size 1.6 1.6) (drill 1.0) (layers "*.Cu" "*.Mask") (remove_unused_layers no) (net 1 "HCP_GND"))
+    (pad "2" thru_hole circle (at -1.53 8.3) (size 1.6 1.6) (drill 1.0) (layers "*.Cu" "*.Mask") (remove_unused_layers no) (net 1 "HCP_GND"))
+    (pad "3" thru_hole circle (at -0.51 10.84) (size 1.6 1.6) (drill 1.0) (layers "*.Cu" "*.Mask") (remove_unused_layers no) (net 4 "HCP_B_MINUS"))
+    (pad "4" thru_hole circle (at 0.51 8.3) (size 1.6 1.6) (drill 1.0) (layers "*.Cu" "*.Mask") (remove_unused_layers no) (net 3 "HCP_A_PLUS"))
+    (pad "5" thru_hole circle (at 1.53 10.84) (size 1.6 1.6) (drill 1.0) (layers "*.Cu" "*.Mask") (remove_unused_layers no) (net 2 "HCP_25V"))
+    (pad "6" thru_hole circle (at 2.55 8.3) (size 1.6 1.6) (drill 1.0) (layers "*.Cu" "*.Mask") (remove_unused_layers no) (net 2 "HCP_25V"))
     (pad "" np_thru_hole circle (at -6.0 6.0) (size 2.5 2.5) (drill 2.5) (layers "*.Cu" "*.Mask"))
     (pad "" np_thru_hole circle (at 6.0 6.0) (size 2.5 2.5) (drill 2.5) (layers "*.Cu" "*.Mask"))
@@
     (embedded_fonts no)
   )
-  (segment (start 127.55 78.84) (end 127.55 77.6) (width 0.5) (layer "F.Cu") (net 2))
-  (segment (start 127.55 77.6) (end 126.53 76.58) (width 0.5) (layer "F.Cu") (net 2))
-  (segment (start 126.53 76.58) (end 126.53 76.3) (width 0.5) (layer "F.Cu") (net 2))
-  (segment (start 126.53 76.3) (end 126.53 71.5) (width 0.8) (layer "F.Cu") (net 2))
-  (segment (start 126.53 71.5) (end 134.75 71.5) (width 0.8) (layer "F.Cu") (net 2))
-  (segment (start 122.45 76.3) (end 122.45 77.82) (width 0.5) (layer "B.Cu") (net 1))
-  (segment (start 122.45 77.82) (end 123.47 78.84) (width 0.5) (layer "B.Cu") (net 1))
-  (segment (start 123.47 78.84) (end 123.47 82.5) (width 0.8) (layer "B.Cu") (net 1))
+  (segment (start 126.53 78.84) (end 127.55 77.82) (width 0.5) (layer "F.Cu") (net 2))
+  (segment (start 127.55 77.82) (end 127.55 76.3) (width 0.5) (layer "F.Cu") (net 2))
+  (segment (start 127.55 76.3) (end 127.55 71.5) (width 0.8) (layer "F.Cu") (net 2))
+  (segment (start 127.55 71.5) (end 134.75 71.5) (width 0.8) (layer "F.Cu") (net 2))
+  (segment (start 123.47 76.3) (end 123.47 77.82) (width 0.5) (layer "B.Cu") (net 1))
+  (segment (start 123.47 77.82) (end 122.45 78.84) (width 0.5) (layer "B.Cu") (net 1))
+  (segment (start 122.45 78.84) (end 122.45 80.4) (width 0.5) (layer "B.Cu") (net 1))
+  (segment (start 122.45 80.4) (end 123.47 81.4) (width 0.5) (layer "B.Cu") (net 1))
+  (segment (start 123.47 81.4) (end 123.47 82.5) (width 0.8) (layer "B.Cu") (net 1))
   (segment (start 123.47 82.5) (end 134.75 82.5) (width 0.8) (layer "B.Cu") (net 1))
   (segment (start 134.75 82.5) (end 134.75 89.0) (width 0.8) (layer "B.Cu") (net 1))
@@
   (segment (start 160.51 103.27) (end 154.5 103.27) (width 0.5) (layer "B.Cu") (net 8))
   (segment (start 154.5 103.27) (end 152.5 103.27) (width 0.5) (layer "F.Cu") (net 8))
-  (segment (start 124.49 76.3) (end 124.49 74.8) (width 0.5) (layer "F.Cu") (net 4))
-  (segment (start 124.49 74.8) (end 121.0 74.8) (width 0.5) (layer "F.Cu") (net 4))
-  (segment (start 121.0 74.8) (end 121.0 80.5) (width 0.5) (layer "F.Cu") (net 4))
-  (segment (start 121.0 80.5) (end 122.0 81.5) (width 0.5) (layer "F.Cu") (net 4))
-  (segment (start 122.0 81.5) (end 122.0 100.5) (width 0.5) (layer "F.Cu") (net 4))
-  (segment (start 122.0 100.5) (end 120.5 102.0) (width 0.5) (layer "F.Cu") (net 4))
+  (segment (start 124.49 78.84) (end 124.49 81.5) (width 0.5) (layer "F.Cu") (net 4))
+  (segment (start 124.49 81.5) (end 122.5 81.5) (width 0.5) (layer "F.Cu") (net 4))
+  (segment (start 122.5 81.5) (end 122.5 100.5) (width 0.5) (layer "F.Cu") (net 4))
+  (segment (start 122.5 100.5) (end 120.5 102.0) (width 0.5) (layer "F.Cu") (net 4))
   (segment (start 120.5 102.0) (end 118.5 102.0) (width 0.5) (layer "F.Cu") (net 4))
-  (segment (start 125.51 78.84) (end 125.51 82.0) (width 0.5) (layer "F.Cu") (net 3))
-  (segment (start 125.51 82.0) (end 124.0 82.0) (width 0.5) (layer "F.Cu") (net 3))
-  (segment (start 124.0 82.0) (end 124.0 107.08) (width 0.5) (layer "F.Cu") (net 3))
-  (segment (start 124.0 107.08) (end 118.5 107.08) (width 0.5) (layer "F.Cu") (net 3))
+  (segment (start 125.51 76.3) (end 125.51 74.8) (width 0.5) (layer "B.Cu") (net 3))
+  (segment (start 125.51 74.8) (end 121.0 74.8) (width 0.5) (layer "B.Cu") (net 3))
+  (segment (start 121.0 74.8) (end 121.0 80.5) (width 0.5) (layer "B.Cu") (net 3))
+  (segment (start 121.0 80.5) (end 122.0 81.5) (width 0.5) (layer "B.Cu") (net 3))
+  (segment (start 122.0 81.5) (end 122.0 107.08) (width 0.5) (layer "B.Cu") (net 3))
+  (segment (start 122.0 107.08) (end 118.5 107.08) (width 0.5) (layer "F.Cu") (net 3))
   (via (at 154.5 103.27) (size 0.8) (drill 0.4) (layers "F.Cu" "B.Cu") (net 8))
+  (via (at 122.0 107.08) (size 0.8) (drill 0.4) (layers "F.Cu" "B.Cu") (net 3))
   (gr_rect (start 116.0 68.0) (end 181.0 112.5) (stroke (width 0.1) (type default)) (fill none) (layer "Edge.Cuts"))
   (gr_line (start 179.0 83.3) (end 179.0 80.6) (stroke (width 0.2) (type default)) (layer "F.SilkS"))
@@
   (gr_text "Hörmann" (at 126.8 82.6 0) (layer "F.SilkS") (effects (font (size 0.8 0.8) (thickness 0.15))))
   (gr_text "HCP2 Adapter" (at 126.8 84.0 0) (layer "F.SilkS") (effects (font (size 0.8 0.8) (thickness 0.15))))
-  (gr_text "5bc247c" (at 126.8 85.4 0) (layer "F.SilkS") (effects (font (size 0.8 0.8) (thickness 0.15))))
+  (gr_text "f21ee3d" (at 126.8 85.4 0) (layer "F.SilkS") (effects (font (size 0.8 0.8) (thickness 0.15))))
   (gr_text "(C) 2026" (at 126.8 86.8 0) (layer "F.SilkS") (effects (font (size 0.8 0.8) (thickness 0.15))))
   (gr_text "Thies Gerken" (at 126.8 88.2 0) (layer "F.SilkS") (effects (font (size 0.8 0.8) (thickness 0.15))))
-  (gr_text "1" (at 122.45 80.6 0) (layer "F.SilkS") (effects (font (size 0.8 0.8) (thickness 0.15))))
+  (gr_text "1" (at 120.9 78.84 0) (layer "F.SilkS") (effects (font (size 0.8 0.8) (thickness 0.15))))
   (gr_text "!" (at 177.5 82.0 0) (layer "F.SilkS") (effects (font (size 1.4 1.4) (thickness 0.25))))
   (gr_text "DISCONNECT" (at 178.4 88.2 90) (layer "F.SilkS") (effects (font (size 0.8 0.8) (thickness 0.15))))
