File: hardware/pcb/generated/hcp.kicad_pcb (KiCad board)
At the start: 2 copper layers, 65 x 44.5 mm, 9 parts, among them J1 HCP2 6P6C, U1 ESP32-C3 Super Mini, U2 Isolated RS485

Commit message: Regenerate outputs
Co-Authored-By: Claude Fable 5.1 <noreply@anthropic.com>
Routing:
- net HCP_25V: track 15.0 -> 20.1 mm
- net HCP_GND: track 109.9 -> 105.4 mm
- net HCP_B_MINUS: track 28.1 -> 29.2 mm
- net HCP_A_PLUS: track 42.2 -> 41.2 mm
Other:
- board text added: "7f6d307"
- board text removed: "f21ee3d"
Changed lines of the file:
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@@
     (layer "F.Cu")
     (at 125.0 68.0 0)
-    (descr "95001-type 6P6C modular jack, side entry, front face flush with the board edge. Pegs 2.4 mm at 12.0 mm, pins 1.02 mm stagger in rows 8.3/10.84 mm behind the edge, odd pins in the rear row. From vendor drawings, verify on delivered part.")
+    (descr "95001-type 6P6C modular jack, side entry, front face flush with the board edge. Pegs 2.4 mm at 12.0 mm, latch down, pin 1 right rear in top view, pins alternate rear/front. Pegs and rows from family drawings, orientation from the vendor photo, verify on delivered part.")
     (tags "RJ12 RJ11 6P6C 95001")
     (property "Reference" "J1" (at 0.00 3.00 0) (layer "F.SilkS") (effects (font (size 1.0 1.0) (thickness 0.15))))
@@
     (property "Description" "" (at 0 0 0) (layer "F.Fab") (hide yes) (effects (font (size 1.0 1.0) (thickness 0.15))))
     (attr through_hole)
-    (pad "1" thru_hole rect (at -2.55 10.84) (size 1.6 1.6) (drill 1.0) (layers "*.Cu" "*.Mask") (remove_unused_layers no) (net 1 "HCP_GND"))
-    (pad "2" thru_hole circle (at -1.53 8.3) (size 1.6 1.6) (drill 1.0) (layers "*.Cu" "*.Mask") (remove_unused_layers no) (net 1 "HCP_GND"))
-    (pad "3" thru_hole circle (at -0.51 10.84) (size 1.6 1.6) (drill 1.0) (layers "*.Cu" "*.Mask") (remove_unused_layers no) (net 4 "HCP_B_MINUS"))
-    (pad "4" thru_hole circle (at 0.51 8.3) (size 1.6 1.6) (drill 1.0) (layers "*.Cu" "*.Mask") (remove_unused_layers no) (net 3 "HCP_A_PLUS"))
-    (pad "5" thru_hole circle (at 1.53 10.84) (size 1.6 1.6) (drill 1.0) (layers "*.Cu" "*.Mask") (remove_unused_layers no) (net 2 "HCP_25V"))
-    (pad "6" thru_hole circle (at 2.55 8.3) (size 1.6 1.6) (drill 1.0) (layers "*.Cu" "*.Mask") (remove_unused_layers no) (net 2 "HCP_25V"))
+    (pad "1" thru_hole rect (at 2.55 10.84) (size 1.6 1.6) (drill 1.0) (layers "*.Cu" "*.Mask") (remove_unused_layers no) (net 1 "HCP_GND"))
+    (pad "2" thru_hole circle (at 1.53 8.3) (size 1.6 1.6) (drill 1.0) (layers "*.Cu" "*.Mask") (remove_unused_layers no) (net 1 "HCP_GND"))
+    (pad "3" thru_hole circle (at 0.51 10.84) (size 1.6 1.6) (drill 1.0) (layers "*.Cu" "*.Mask") (remove_unused_layers no) (net 4 "HCP_B_MINUS"))
+    (pad "4" thru_hole circle (at -0.51 8.3) (size 1.6 1.6) (drill 1.0) (layers "*.Cu" "*.Mask") (remove_unused_layers no) (net 3 "HCP_A_PLUS"))
+    (pad "5" thru_hole circle (at -1.53 10.84) (size 1.6 1.6) (drill 1.0) (layers "*.Cu" "*.Mask") (remove_unused_layers no) (net 2 "HCP_25V"))
+    (pad "6" thru_hole circle (at -2.55 8.3) (size 1.6 1.6) (drill 1.0) (layers "*.Cu" "*.Mask") (remove_unused_layers no) (net 2 "HCP_25V"))
     (pad "" np_thru_hole circle (at -6.0 6.0) (size 2.5 2.5) (drill 2.5) (layers "*.Cu" "*.Mask"))
     (pad "" np_thru_hole circle (at 6.0 6.0) (size 2.5 2.5) (drill 2.5) (layers "*.Cu" "*.Mask"))
@@
     (embedded_fonts no)
   )
-  (segment (start 126.53 78.84) (end 127.55 77.82) (width 0.5) (layer "F.Cu") (net 2))
-  (segment (start 127.55 77.82) (end 127.55 76.3) (width 0.5) (layer "F.Cu") (net 2))
-  (segment (start 127.55 76.3) (end 127.55 71.5) (width 0.8) (layer "F.Cu") (net 2))
-  (segment (start 127.55 71.5) (end 134.75 71.5) (width 0.8) (layer "F.Cu") (net 2))
-  (segment (start 123.47 76.3) (end 123.47 77.82) (width 0.5) (layer "B.Cu") (net 1))
-  (segment (start 123.47 77.82) (end 122.45 78.84) (width 0.5) (layer "B.Cu") (net 1))
-  (segment (start 122.45 78.84) (end 122.45 80.4) (width 0.5) (layer "B.Cu") (net 1))
-  (segment (start 122.45 80.4) (end 123.47 81.4) (width 0.5) (layer "B.Cu") (net 1))
-  (segment (start 123.47 81.4) (end 123.47 82.5) (width 0.8) (layer "B.Cu") (net 1))
-  (segment (start 123.47 82.5) (end 134.75 82.5) (width 0.8) (layer "B.Cu") (net 1))
-  (segment (start 134.75 82.5) (end 134.75 89.0) (width 0.8) (layer "B.Cu") (net 1))
+  (segment (start 123.47 78.84) (end 122.45 77.82) (width 0.5) (layer "F.Cu") (net 2))
+  (segment (start 122.45 77.82) (end 122.45 76.3) (width 0.5) (layer "F.Cu") (net 2))
+  (segment (start 122.45 76.3) (end 122.45 71.5) (width 0.8) (layer "F.Cu") (net 2))
+  (segment (start 122.45 71.5) (end 134.75 71.5) (width 0.8) (layer "F.Cu") (net 2))
+  (segment (start 126.53 76.3) (end 126.53 77.82) (width 0.5) (layer "F.Cu") (net 1))
+  (segment (start 126.53 77.82) (end 127.55 78.84) (width 0.5) (layer "F.Cu") (net 1))
+  (segment (start 127.55 78.84) (end 127.55 82.5) (width 0.8) (layer "F.Cu") (net 1))
+  (segment (start 127.55 82.5) (end 134.75 82.5) (width 0.8) (layer "F.Cu") (net 1))
+  (segment (start 134.75 82.5) (end 134.75 89.0) (width 0.8) (layer "F.Cu") (net 1))
   (segment (start 134.75 89.0) (end 134.75 91.9) (width 0.8) (layer "F.Cu") (net 1))
   (segment (start 134.75 91.9) (end 174.15 91.9) (width 0.8) (layer "F.Cu") (net 1))
@@
   (segment (start 160.51 103.27) (end 154.5 103.27) (width 0.5) (layer "B.Cu") (net 8))
   (segment (start 154.5 103.27) (end 152.5 103.27) (width 0.5) (layer "F.Cu") (net 8))
-  (segment (start 124.49 78.84) (end 124.49 81.5) (width 0.5) (layer "F.Cu") (net 4))
-  (segment (start 124.49 81.5) (end 122.5 81.5) (width 0.5) (layer "F.Cu") (net 4))
+  (segment (start 125.51 78.84) (end 125.51 81.5) (width 0.5) (layer "F.Cu") (net 4))
+  (segment (start 125.51 81.5) (end 122.5 81.5) (width 0.5) (layer "F.Cu") (net 4))
   (segment (start 122.5 81.5) (end 122.5 100.5) (width 0.5) (layer "F.Cu") (net 4))
   (segment (start 122.5 100.5) (end 120.5 102.0) (width 0.5) (layer "F.Cu") (net 4))
   (segment (start 120.5 102.0) (end 118.5 102.0) (width 0.5) (layer "F.Cu") (net 4))
-  (segment (start 125.51 76.3) (end 125.51 74.8) (width 0.5) (layer "B.Cu") (net 3))
-  (segment (start 125.51 74.8) (end 121.0 74.8) (width 0.5) (layer "B.Cu") (net 3))
+  (segment (start 124.49 76.3) (end 124.49 74.8) (width 0.5) (layer "B.Cu") (net 3))
+  (segment (start 124.49 74.8) (end 121.0 74.8) (width 0.5) (layer "B.Cu") (net 3))
   (segment (start 121.0 74.8) (end 121.0 80.5) (width 0.5) (layer "B.Cu") (net 3))
   (segment (start 121.0 80.5) (end 122.0 81.5) (width 0.5) (layer "B.Cu") (net 3))
@@
   (gr_text "Hörmann" (at 126.8 82.6 0) (layer "F.SilkS") (effects (font (size 0.8 0.8) (thickness 0.15))))
   (gr_text "HCP2 Adapter" (at 126.8 84.0 0) (layer "F.SilkS") (effects (font (size 0.8 0.8) (thickness 0.15))))
-  (gr_text "f21ee3d" (at 126.8 85.4 0) (layer "F.SilkS") (effects (font (size 0.8 0.8) (thickness 0.15))))
+  (gr_text "7f6d307" (at 126.8 85.4 0) (layer "F.SilkS") (effects (font (size 0.8 0.8) (thickness 0.15))))
   (gr_text "(C) 2026" (at 126.8 86.8 0) (layer "F.SilkS") (effects (font (size 0.8 0.8) (thickness 0.15))))
   (gr_text "Thies Gerken" (at 126.8 88.2 0) (layer "F.SilkS") (effects (font (size 0.8 0.8) (thickness 0.15))))
-  (gr_text "1" (at 120.9 78.84 0) (layer "F.SilkS") (effects (font (size 0.8 0.8) (thickness 0.15))))
+  (gr_text "1" (at 129.1 78.84 0) (layer "F.SilkS") (effects (font (size 0.8 0.8) (thickness 0.15))))
   (gr_text "!" (at 177.5 82.0 0) (layer "F.SilkS") (effects (font (size 1.4 1.4) (thickness 0.25))))
   (gr_text "DISCONNECT" (at 178.4 88.2 90) (layer "F.SilkS") (effects (font (size 0.8 0.8) (thickness 0.15))))

Commit message: Regenerate outputs
Co-Authored-By: Claude Fable 5.1 <noreply@anthropic.com>
Parts:
- J1: footprint HCP:RJ12_95001_6P6C -> HCP:RJ12_Amphenol_54601-x06_Horizontal
- moved J1 17.1 mm to (128.2, 84.8), turned to 180 degrees
- moved H1 5.00 mm to (119.5, 89.5)
Routing:
- net HCP_GND: track 105.4 -> 98.9 mm
- net HCP_25V: track 20.1 -> 26.3 mm
- net HCP_B_MINUS: track 29.2 -> 23.4 mm
- net HCP_A_PLUS: track 41.2 -> 37.0 mm
Other:
- board text added: "Adapter 004133b"
- board text added: "Hörmann HCP2"
- board text removed: "7f6d307"
- board text removed: "HCP2 Adapter"
- board text removed: "Hörmann"

Commit message: Regenerate outputs
Co-Authored-By: Claude Fable 5.1 <noreply@anthropic.com>
Parts:
- removed H2: M3, HCP:MountingHole_3.2mm_NoCourtyard
- moved H3 1.00 mm to (154.9, 108.5)
Other:
- board text added: "Adapter 54eaa7b"
- board text removed: "Adapter 004133b"
Changed lines of the file:
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@@
   (footprint "HCP:MountingHole_3.2mm_NoCourtyard"
     (layer "F.Cu")
-    (at 178.2 71.5 0)
-    (descr "M3 mounting hole without courtyard, for placement under socketed modules")
-    (tags "mounting hole M3")
-    (property "Reference" "H2" (at 0 -3 0) (layer "F.SilkS") (hide yes) (effects (font (size 1.0 1.0) (thickness 0.15))))
-    (property "Value" "M3" (at 0 3 0) (layer "F.Fab") (hide yes) (effects (font (size 1.0 1.0) (thickness 0.15))))
-    (property "Datasheet" "" (at 0 0 0) (layer "F.Fab") (hide yes) (effects (font (size 1.0 1.0) (thickness 0.15))))
-    (property "Description" "" (at 0 0 0) (layer "F.Fab") (hide yes) (effects (font (size 1.0 1.0) (thickness 0.15))))
-    (attr exclude_from_pos_files exclude_from_bom)
-    (pad "" np_thru_hole circle (at 0 0) (size 3.2 3.2) (drill 3.2) (layers "*.Cu" "*.Mask"))
-    (embedded_fonts no)
-  )
-  (footprint "HCP:MountingHole_3.2mm_NoCourtyard"
-    (layer "F.Cu")
-    (at 155.9 108.5 0)
+    (at 154.9 108.5 0)
     (descr "M3 mounting hole without courtyard, for placement under socketed modules")
     (tags "mounting hole M3")
@@
   (gr_line (start 179.0 80.6) (end 179.6 81.4) (stroke (width 0.2) (type default)) (layer "F.SilkS"))
   (gr_text "Hörmann HCP2" (at 127.4 87.2 0) (layer "F.SilkS") (effects (font (size 0.8 0.8) (thickness 0.15))))
-  (gr_text "Adapter 004133b" (at 127.4 88.6 0) (layer "F.SilkS") (effects (font (size 0.8 0.8) (thickness 0.15))))
+  (gr_text "Adapter 54eaa7b" (at 127.4 88.6 0) (layer "F.SilkS") (effects (font (size 0.8 0.8) (thickness 0.15))))
   (gr_text "(C) 2026" (at 127.4 90.0 0) (layer "F.SilkS") (effects (font (size 0.8 0.8) (thickness 0.15))))
   (gr_text "Thies Gerken" (at 127.4 91.4 0) (layer "F.SilkS") (effects (font (size 0.8 0.8) (thickness 0.15))))
