File: hardware/pcb/generated/hcp.kicad_sch (KiCad schematic)
At the start: 5 parts, among them J1 HCP2 6P6C, U1 ESP32-C3 Super Mini, U2 Isolated RS485, auto directio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

Commit message: Regenerate outputs
Co-Authored-By: Claude Fable 5.1 <noreply@anthropic.com>
Parts:
- J1: footprint HCP:RJ12_95001_6P6C -> HCP:RJ12_Amphenol_54601-x06_Horizontal
Changed lines of the file:
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@@
 (kicad_sch (version 20231120) (generator "hoermann-schematic") (generator_version "1")
   (paper "A4")
-  (title_block (title "Hörmann HCP2 ESP32-C3 Adapter") (date "2026-09-05") (rev "7f6d307") (company "Thies Gerken"))
+  (title_block (title "Hörmann HCP2 ESP32-C3 Adapter") (date "2026-09-05") (rev "004133b") (company "Thies Gerken"))
   (symbol (lib_id "HCP:J1") (at 40.64 88.9 0) (unit 1) (exclude_from_sim no) (in_bom yes) (on_board yes) (dnp no)
     (property "Reference" "J1" (at 40.64 78.74 0) (effects (font (size 1.27 1.27))))
     (property "Value" "HCP2 6P6C" (at 40.64 99.06 0) (effects (font (size 1.27 1.27))))
-    (property "Footprint" "HCP:RJ12_95001_6P6C" (at 40.64 88.9 0) (effects (font (size 1.27 1.27)) (hide yes)))
+    (property "Footprint" "HCP:RJ12_Amphenol_54601-x06_Horizontal" (at 40.64 88.9 0) (effects (font (size 1.27 1.27)) (hide yes)))
     (property "Datasheet" "" (at 40.64 88.9 0) (effects (font (size 1.27 1.27)) (hide yes)))
     (pin "6")
