File: pcb/hcp.kicad_pcb (KiCad board)
At the start: 2 copper layers, 65 x 44.5 mm, 8 parts, among them J1 HCP2 6P6C, U1 ESP32-C3 Super Mini, U2 Isolated RS485

Commit message: Flatten project outputs and refine README
Other:
- board text added: "Adapter 609722a"
- board text removed: "Adapter 977c400"
Changed lines of the file:
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@@
   (gr_line (start 179.0 80.6) (end 179.6 81.4) (stroke (width 0.2) (type default)) (layer "F.SilkS"))
   (gr_text "Hörmann HCP2" (at 127.4 87.2 0) (layer "F.SilkS") (effects (font (size 0.8 0.8) (thickness 0.15))))
-  (gr_text "Adapter 977c400" (at 127.4 88.6 0) (layer "F.SilkS") (effects (font (size 0.8 0.8) (thickness 0.15))))
+  (gr_text "Adapter 609722a" (at 127.4 88.6 0) (layer "F.SilkS") (effects (font (size 0.8 0.8) (thickness 0.15))))
   (gr_text "(C) 2026" (at 127.4 90.0 0) (layer "F.SilkS") (effects (font (size 0.8 0.8) (thickness 0.15))))
   (gr_text "Thies Gerken" (at 127.4 91.4 0) (layer "F.SilkS") (effects (font (size 0.8 0.8) (thickness 0.15))))
