File: pcb/hcp.kicad_pcb (KiCad board)
At the start: 2 copper layers, 65 x 44.5 mm, 8 parts, among them J1 HCP2 6P6C, U1 ESP32-C3 Super Mini, U2 Isolated RS485

Commit message: Correct the UART pin roles against the RS485 module
The module names its TTL pads from its own point of view, so the pad marked
TX is the receiver output that drives the MCU. Wiring the ESP32 transmitter
to it left the RS485 driver permanently off, which is why the adapter never
registered on the bus.

The copper is unaffected, only the net names, the symbol pin directions and
the ESPHome pin assignment change. Confirmed on the assembled board: A/B move
from the 185 mV idle bias to 1.62 V under transmit load, and the opener now
polls the adapter continuously.

Co-Authored-By: Claude Opus 5 <noreply@anthropic.com>
Connections:
- net UART_RX_GPIO20 renamed UART_TX_GPIO20
- net UART_TX_GPIO21 renamed UART_RX_GPIO21
Other:
- board text added: "Adapter 32cfca7"
- board text removed: "Adapter 609722a"
Changed lines of the file:
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@@
   (net 6 "ESP_5V")
   (net 7 "ESP_3V3")
-  (net 8 "UART_TX_GPIO21")
-  (net 9 "UART_RX_GPIO20")
+  (net 8 "UART_RX_GPIO21")
+  (net 9 "UART_TX_GPIO20")
   (footprint "HCP:RJ12_Amphenol_54601-x06_Horizontal"
   	(layer "F.Cu")
@@
     (fp_text user "IO10" (at -5.6 3.81 0) (layer "F.Fab") (effects (font (size 0.6 0.6) (thickness 0.10))))
     (pad "13" thru_hole circle (at 7.62 6.35 270) (size 1.7 1.7) (drill 1.0) (layers "*.Cu" "*.Mask") (remove_unused_layers no))
-    (pad "14" thru_hole circle (at -7.62 6.35 270) (size 1.7 1.7) (drill 1.0) (layers "*.Cu" "*.Mask") (remove_unused_layers no) (net 9 "UART_RX_GPIO20"))
+    (pad "14" thru_hole circle (at -7.62 6.35 270) (size 1.7 1.7) (drill 1.0) (layers "*.Cu" "*.Mask") (remove_unused_layers no) (net 9 "UART_TX_GPIO20"))
     (fp_text user "IO1" (at 5.6 6.35 0) (layer "F.Fab") (effects (font (size 0.6 0.6) (thickness 0.10))))
     (fp_text user "IO20" (at -5.6 6.35 0) (layer "F.Fab") (effects (font (size 0.6 0.6) (thickness 0.10))))
     (pad "15" thru_hole circle (at 7.62 8.89 270) (size 1.7 1.7) (drill 1.0) (layers "*.Cu" "*.Mask") (remove_unused_layers no))
-    (pad "16" thru_hole circle (at -7.62 8.89 270) (size 1.7 1.7) (drill 1.0) (layers "*.Cu" "*.Mask") (remove_unused_layers no) (net 8 "UART_TX_GPIO21"))
+    (pad "16" thru_hole circle (at -7.62 8.89 270) (size 1.7 1.7) (drill 1.0) (layers "*.Cu" "*.Mask") (remove_unused_layers no) (net 8 "UART_RX_GPIO21"))
     (fp_text user "IO0" (at 5.6 8.89 0) (layer "F.Fab") (effects (font (size 0.6 0.6) (thickness 0.10))))
     (fp_text user "IO21" (at -5.6 8.89 0) (layer "F.Fab") (effects (font (size 0.6 0.6) (thickness 0.10))))
@@
     (pad "1" smd roundrect (at -17 -3.81 180) (size 2.4 2.0) (layers "F.Cu" "F.Paste" "F.Mask") (roundrect_rratio 0.2) (net 7 "ESP_3V3"))
     (fp_text user "VIN" (at -14.4 -3.81 0) (layer "F.Fab") (effects (font (size 0.6 0.6) (thickness 0.10))))
-    (pad "2" smd roundrect (at -17 -1.27 180) (size 2.4 2.0) (layers "F.Cu" "F.Paste" "F.Mask") (roundrect_rratio 0.2) (net 8 "UART_TX_GPIO21"))
+    (pad "2" smd roundrect (at -17 -1.27 180) (size 2.4 2.0) (layers "F.Cu" "F.Paste" "F.Mask") (roundrect_rratio 0.2) (net 8 "UART_RX_GPIO21"))
     (fp_text user "TX" (at -14.4 -1.27 0) (layer "F.Fab") (effects (font (size 0.6 0.6) (thickness 0.10))))
-    (pad "3" smd roundrect (at -17 1.27 180) (size 2.4 2.0) (layers "F.Cu" "F.Paste" "F.Mask") (roundrect_rratio 0.2) (net 9 "UART_RX_GPIO20"))
+    (pad "3" smd roundrect (at -17 1.27 180) (size 2.4 2.0) (layers "F.Cu" "F.Paste" "F.Mask") (roundrect_rratio 0.2) (net 9 "UART_TX_GPIO20"))
     (fp_text user "RX" (at -14.4 1.27 0) (layer "F.Fab") (effects (font (size 0.6 0.6) (thickness 0.10))))
     (pad "4" smd roundrect (at -17 3.81 180) (size 2.4 2.0) (layers "F.Cu" "F.Paste" "F.Mask") (roundrect_rratio 0.2) (net 1 "HCP_GND"))
@@
   (gr_line (start 179.0 80.6) (end 179.6 81.4) (stroke (width 0.2) (type default)) (layer "F.SilkS"))
   (gr_text "Hörmann HCP2" (at 127.4 87.2 0) (layer "F.SilkS") (effects (font (size 0.8 0.8) (thickness 0.15))))
-  (gr_text "Adapter 609722a" (at 127.4 88.6 0) (layer "F.SilkS") (effects (font (size 0.8 0.8) (thickness 0.15))))
+  (gr_text "Adapter 32cfca7" (at 127.4 88.6 0) (layer "F.SilkS") (effects (font (size 0.8 0.8) (thickness 0.15))))
   (gr_text "(C) 2026" (at 127.4 90.0 0) (layer "F.SilkS") (effects (font (size 0.8 0.8) (thickness 0.15))))
   (gr_text "Thies Gerken" (at 127.4 91.4 0) (layer "F.SilkS") (effects (font (size 0.8 0.8) (thickness 0.15))))
