File: pcb/hcp.kicad_sch (KiCad schematic)
At the start: 5 parts, among them J1 HCP2 6P6C, U1 ESP32-C3 Super Mini, U2 Isolated RS485, auto directio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

Commit message: Correct the UART pin roles against the RS485 module
The module names its TTL pads from its own point of view, so the pad marked
TX is the receiver output that drives the MCU. Wiring the ESP32 transmitter
to it left the RS485 driver permanently off, which is why the adapter never
registered on the bus.

The copper is unaffected, only the net names, the symbol pin directions and
the ESPHome pin assignment change. Confirmed on the assembled board: A/B move
from the 185 mV idle bias to 1.62 V under transmit load, and the opener now
polls the adapter continuously.

Co-Authored-By: Claude Opus 5 <noreply@anthropic.com>
Connections:
- net UART_RX_GPIO20 renamed UART_TX_GPIO20
- net UART_TX_GPIO21 renamed UART_RX_GPIO21
Other:
- note added: "U2 is powered from 3V3 so its TX output stays at ESP32 logic level."
- note added: "U2 pin names are from the module's own view: TX drives the ESP32, RX is driven by it."
- note removed: "U2 is powered from 3V3 so its RX output stays at ESP32 logic level."
Changed lines of the file:
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@@
 (kicad_sch (version 20231120) (generator "hoermann-schematic") (generator_version "1")
   (paper "A4")
-  (title_block (title "Hörmann HCP2 ESP32-C3 Adapter") (date "2026-09-05") (rev "609722a") (company "Thies Gerken"))
+  (title_block (title "Hörmann HCP2 ESP32-C3 Adapter") (date "2026-09-05") (rev "32cfca7") (company "Thies Gerken"))
   (symbol (lib_id "HCP:J1") (at 40.64 88.9 0) (unit 1) (exclude_from_sim no) (in_bom yes) (on_board yes) (dnp no)
     (property "Reference" "J1" (at 40.64 78.74 0) (effects (font (size 1.27 1.27))))
@@
   (label "ESP_5V" (at 185.42 78.74 90) (fields_autoplaced yes) (effects (font (size 1.27 1.27)) (justify left bottom)))
   (label "ESP_3V3" (at 152.4 110.49 0) (fields_autoplaced yes) (effects (font (size 1.27 1.27)) (justify left bottom)))
-  (label "UART_TX_GPIO21" (at 152.4 113.03 0) (fields_autoplaced yes) (effects (font (size 1.27 1.27)) (justify left bottom)))
-  (label "UART_RX_GPIO20" (at 152.4 115.57 0) (fields_autoplaced yes) (effects (font (size 1.27 1.27)) (justify left bottom)))
+  (label "UART_RX_GPIO21" (at 152.4 113.03 0) (fields_autoplaced yes) (effects (font (size 1.27 1.27)) (justify left bottom)))
+  (label "UART_TX_GPIO20" (at 152.4 115.57 0) (fields_autoplaced yes) (effects (font (size 1.27 1.27)) (justify left bottom)))
   (no_connect (at 99.06 119.38))
   (no_connect (at 226.06 95.25))
@@
   (text "HCP2 bus, 6P6C. Contact numbering per ESPHome HCP documentation." (exclude_from_sim no) (at 25.4 128.27 0) (effects (font (size 1.27 1.27)) (justify left bottom)))
   (text "Adjust PS1 to 5.0 V before connecting U1. Open JP1 whenever USB is plugged into U1." (exclude_from_sim no) (at 99.06 45.72 0) (effects (font (size 1.27 1.27)) (justify left bottom)))
-  (text "U2 is powered from 3V3 so its RX output stays at ESP32 logic level." (exclude_from_sim no) (at 99.06 132.08 0) (effects (font (size 1.27 1.27)) (justify left bottom)))
+  (text "U2 is powered from 3V3 so its TX output stays at ESP32 logic level." (exclude_from_sim no) (at 99.06 132.08 0) (effects (font (size 1.27 1.27)) (justify left bottom)))
+  (text "U2 pin names are from the module's own view: TX drives the ESP32, RX is driven by it." (exclude_from_sim no) (at 99.06 135.89 0) (effects (font (size 1.27 1.27)) (justify left bottom)))
   (sheet_instances (path "/" (page "1")))
 )
